Commit message: Adding gazebo launch files

File: viratsim/description/virat_description.urdf.xacro (robot description, xacro)
@@ -1,4 +1,4 @@
 <?xml version="1.0"?>
-<robot name="virat" xmlns:xacro="http://ros.org/wiki/xacro">
+<robot name="virat" xmlns:xacro="http://ros.org/wiki/xacro">>
 	<link name="body">
 		<visual>
@@ -8,14 +8,4 @@
 			<origin rpy="0.0 0 0" xyz="0 0 0"/>
 		</visual>
-		<collision>
-			<geometry>
-				<box size="0.75 1 1">
-        		</geometry>
-			<origin rpy="0.0 0 0" xyz="0 0 0"/>
-		</collision>
-		<inertial>
-			<mass value="0.5"/>
-			<inertia ixx="1.0" ixy="0.0" ixz="0.0" iyy="1.0" iyz="0.0" izz="1.0" />
-		</inertial>
 	</link>
 	<link name="front_wheel">
@@ -26,10 +16,4 @@
         		</geometry>
 		</visual>
-        	<collision>
-			<geometry>
-				<box size="0.1 0.2 0.2"/>
-        		</geometry>
-			<origin rpy="0.0 0 0" xyz="0 0 0"/>
-		</collision>
 	</link>
 	<joint name="front_axle" type="continuous">
@@ -45,10 +29,4 @@
         		</geometry>
 		</visual>
-		<collision>
-			<geometry>
-				<box size="0.1 0.2 0.05"/>
-        		</geometry>
-			<origin rpy="0.0 0 0" xyz="0 0 0"/>
-		</collision>
 	</link>
 	<joint name="rear_axle" type="continuous">

Commit message: Added proper collision and inertial tags to the urdf. GAZEBO LAUNCH WORKS!!!! (YAAAAYYYYY!!!!)

File: viratsim/description/virat_description.urdf.xacro (robot description, xacro)
@@ -1,11 +1,29 @@
 <?xml version="1.0"?>
-<robot name="virat" xmlns:xacro="http://ros.org/wiki/xacro">>
+<robot name="virat" xmlns:xacro="http://ros.org/wiki/xacro">
+	<xacro:macro name="default_inertial" params="mass">
+		<inertial>
+			<origin rpy="0.0 0 0" xyz="0 0 0"/>
+			<mass value="${mass}" />
+			<inertia ixx="1.0" ixy="0.0" ixz="0.0" iyy="1.0" iyz="0.0" izz="1.0" />
+		</inertial>
+	</xacro:macro>
+	<material name="white">
+		<color rgba="1 1 1 1"/>
+	</material>
 	<link name="body">
 		<visual>
+			<origin rpy="0.0 0 0" xyz="0 0 0"/>
 			<geometry>
 				<mesh filename="package://viratsim/meshes/body/bot2.dae"/>
         		</geometry>
+			<material name="white"/>
+		</visual>
+		<collision>
 			<origin rpy="0.0 0 0" xyz="0 0 0"/>
-		</visual>
+			<geometry>
+				<mesh filename="package://viratsim/meshes/body/bot2.dae"/>
+			</geometry>
+		</collision>
+		<xacro:default_inertial mass="50"/>
 	</link>
 	<link name="front_wheel">
@@ -15,5 +33,13 @@
 				<mesh filename="package://viratsim/meshes/wheels/castors1.dae"/>
         		</geometry>
+        		<material name="white"/>
 		</visual>
+		<collision>
+			<origin rpy="0.0 0 0" xyz="0.5 0 0"/>
+			<geometry>
+				<mesh filename="package://viratsim/meshes/wheels/castors1.dae"/>
+        		</geometry>
+		</collision>
+		<xacro:default_inertial mass="1"/>
 	</link>
 	<joint name="front_axle" type="continuous">
@@ -28,5 +54,13 @@
 				<mesh filename="package://viratsim/meshes/wheels/tyre1.dae"/>
         		</geometry>
+        		<material name="white"/>
 		</visual>
+		<collision>
+			<origin rpy="0.0 0 0" xyz="0 0 0"/>
+			<geometry>
+				<mesh filename="package://viratsim/meshes/wheels/tyre1.dae"/>
+        		</geometry>
+		</collision>
+		<xacro:default_inertial mass="5"/>
 	</link>
 	<joint name="rear_axle" type="continuous">

Commit message: attached joints,pls figure out ryp

File: viratsim/description/virat_description.urdf.xacro (robot description, xacro)
@@ -13,5 +13,5 @@
 	<link name="body">
 		<visual>
-			<origin rpy="0.0 0 0" xyz="0 0 0"/>
+			<origin  xyz="0 0 0"/>
 			<geometry>
 				<mesh filename="package://viratsim/meshes/body/bot2.dae"/>
@@ -20,5 +20,5 @@
 		</visual>
 		<collision>
-			<origin rpy="0.0 0 0" xyz="0 0 0"/>
+			<origin  xyz="0 0 0"/>
 			<geometry>
 				<mesh filename="package://viratsim/meshes/body/bot2.dae"/>
@@ -29,5 +29,5 @@
 	<link name="front_wheel">
 		<visual>
-			<origin rpy="0.0 0 0" xyz="0.5 0 0"/>
+			<origin  xyz="0 0 0"/>
 			<geometry>
 				<mesh filename="package://viratsim/meshes/wheels/castors1.dae"/>
@@ -36,5 +36,5 @@
 		</visual>
 		<collision>
-			<origin rpy="0.0 0 0" xyz="0.5 0 0"/>
+			<origin  xyz="0 0 0"/>
 			<geometry>
 				<mesh filename="package://viratsim/meshes/wheels/castors1.dae"/>
@@ -46,9 +46,9 @@
 		<parent link="body"/>
 		<child link="front_wheel"/>
-		<origin xyz="0.5 0 0.05"/>
+		<origin rpy="0 1 0" xyz="0.48 0 0.02"/>
 	</joint>
-	<link name="rear_wheel">
+	<link name="rear_wheel_1">
 		<visual>
-			<origin rpy="0.0 0 0" xyz="0 0 0"/>
+			<origin  xyz="0 0 0"/>
 			<geometry>
 				<mesh filename="package://viratsim/meshes/wheels/tyre1.dae"/>
@@ -57,5 +57,5 @@
 		</visual>
 		<collision>
-			<origin rpy="0.0 0 0" xyz="0 0 0"/>
+			<origin  xyz="0 0 0"/>
 			<geometry>
 				<mesh filename="package://viratsim/meshes/wheels/tyre1.dae"/>
@@ -64,8 +64,29 @@
 		<xacro:default_inertial mass="5"/>
 	</link>
-	<joint name="rear_axle" type="continuous">
+	<joint name="rear_axle_1" type="continuous">
 		<parent link="body"/>
-		<child link="rear_wheel"/>
-		<origin xyz="0 0 0"/>
+		<child link="rear_wheel_1"/>
+		<origin rpy="0 1 0" xyz="0 -0.323 0"/>
+	</joint>
+	<link name="rear_wheel_2">
+		<visual>
+			<origin  xyz="0 0 0"/>
+			<geometry>
+				<mesh filename="package://viratsim/meshes/wheels/tyre1.dae"/>
+        		</geometry>
+        		<material name="white"/>
+		</visual>
+		<collision>
+			<origin  xyz="0 0 0"/>
+			<geometry>
+				<mesh filename="package://viratsim/meshes/wheels/tyre1.dae"/>
+        		</geometry>
+		</collision>
+		<xacro:default_inertial mass="5"/>
+	</link>
+	<joint name="rear_axle_2" type="continuous">
+		<parent link="body"/>
+		<child link="rear_wheel_2"/>
+		<origin rpy="0 1 0" xyz="0 0.323 0"/>
 	</joint>
 </robot>
