Commit message: made world, world launch, fixed axes of wheels.

File: description/virat_description.urdf.xacro (robot description, xacro)
@@ -8,7 +8,4 @@
 		</inertial>
 	</xacro:macro>
-	<material name="white">
-		<color rgba="1 1 1 1"/>
-	</material>
 	<link name="body">
 		<visual>
@@ -17,5 +14,4 @@
 				<mesh filename="package://viratsim/meshes/body/bot2.dae"/>
         		</geometry>
-			<material name="white"/>
 		</visual>
 		<collision>
@@ -33,5 +29,4 @@
 				<mesh filename="package://viratsim/meshes/wheels/castors1.dae"/>
         		</geometry>
-        		<material name="white"/>
 		</visual>
 		<collision>
@@ -46,5 +41,6 @@
 		<parent link="body"/>
 		<child link="front_wheel"/>
-		<origin rpy="0 1 0" xyz="0.48 0 0.02"/>
+		<origin xyz="0.48 0 0.02"/>
+		<axis xyz="0 1 0" rpy="0 0 0"/>
 	</joint>
 	<link name="rear_wheel_1">
@@ -54,5 +50,4 @@
 				<mesh filename="package://viratsim/meshes/wheels/tyre1.dae"/>
         		</geometry>
-        		<material name="white"/>
 		</visual>
 		<collision>
@@ -67,5 +62,6 @@
 		<parent link="body"/>
 		<child link="rear_wheel_1"/>
-		<origin rpy="0 1 0" xyz="0 -0.323 0"/>
+		<origin xyz="0 -0.323 0"/>
+		<axis xyz="0 1 0" rpy="0 0 0"/>
 	</joint>
 	<link name="rear_wheel_2">
@@ -75,5 +71,4 @@
 				<mesh filename="package://viratsim/meshes/wheels/tyre1.dae"/>
         		</geometry>
-        		<material name="white"/>
 		</visual>
 		<collision>
@@ -88,5 +83,6 @@
 		<parent link="body"/>
 		<child link="rear_wheel_2"/>
-		<origin rpy="0 1 0" xyz="0 0.323 0"/>
+		<origin xyz="0 0.323 0"/>
+		<axis xyz="0 1 0" rpy="0 0 0"/>
 	</joint>
 </robot>

Commit message: camera

File: description/virat_description.urdf.xacro (robot description, xacro)
@@ -86,3 +86,57 @@
 		<axis xyz="0 1 0" rpy="0 0 0"/>
 	</joint>
+	<gazebo reference="camera">
+    <sensor type="camera" name="camera">
+      <update_rate>30.0</update_rate>
+      <camera name="head">
+        <horizontal_fov>1.3962634</horizontal_fov>
+        <image>
+          <width>800</width>
+          <height>800</height>
+          <format>R8G8B8</format>
+        </image>
+        <clip>
+          <near>0.02</near>
+          <far>300</far>
+        </clip>
+        <noise>
+          <type>gaussian</type>
+          <mean>0.0</mean>
+          <stddev>0.007</stddev>
+        </noise>
+      </camera>
+      <plugin name="camera_controller" filename="libgazebo_ros_camera.so">
+        <alwaysOn>true</alwaysOn>
+        <updateRate>0.0</updateRate>
+        <cameraName>/mybot/camera</cameraName>
+        <imageTopicName>image_raw</imageTopicName>
+        <cameraInfoTopicName>camera_info</cameraInfoTopicName>
+        <frameName>camera</frameName>
+        <hackBaseline>0.07</hackBaseline>
+        <distortionK1>0.0</distortionK1>
+        <distortionK2>0.0</distortionK2>
+        <distortionK3>0.0</distortionK3>
+        <distortionT1>0.0</distortionT1>
+        <distortionT2>0.0</distortionT2>
+      </plugin>
+    </sensor>
+  </gazebo>
+  <link name="camera">
+    <visual>
+      <geometry>
+        <box size="0.05 0.05 0.05"/>
+      </geometry>
+    </visual>
+    <collision>
+      <geometry>
+        <box size="0.05 0.05 0.05"/>
+      </geometry>
+    </collision>
+    <xacro:default_inertial mass="0.02"/>
+  </link>
+  <joint name="camera_joint" type="fixed">
+    <origin xyz="0.73 0 1.18" rpy="0 0.45 0"/>
+    <parent link="body"/>
+    <child link="camera"/>
+  </joint>
 </robot>

Commit message: added dummy base_link

File: description/virat_description.urdf.xacro (robot description, xacro)
@@ -8,4 +8,5 @@
 		</inertial>
 	</xacro:macro>
+	<link name="base_link"/>
 	<link name="body">
 		<visual>
@@ -23,4 +24,9 @@
 		<xacro:default_inertial mass="50"/>
 	</link>
+	<joint name="dummy_joint" type="fixed">
+		<parent link="base_link"/>
+		<child link="body"/>
+		<origin xyz="0 0 0"/>
+	</joint>
 	<link name="front_wheel">
 		<visual>
@@ -87,56 +93,56 @@
 	</joint>
 	<gazebo reference="camera">
-    <sensor type="camera" name="camera">
-      <update_rate>30.0</update_rate>
-      <camera name="head">
-        <horizontal_fov>1.3962634</horizontal_fov>
-        <image>
-          <width>800</width>
-          <height>800</height>
-          <format>R8G8B8</format>
-        </image>
-        <clip>
-          <near>0.02</near>
-          <far>300</far>
-        </clip>
-        <noise>
-          <type>gaussian</type>
-          <mean>0.0</mean>
-          <stddev>0.007</stddev>
-        </noise>
-      </camera>
-      <plugin name="camera_controller" filename="libgazebo_ros_camera.so">
-        <alwaysOn>true</alwaysOn>
-        <updateRate>0.0</updateRate>
-        <cameraName>/mybot/camera</cameraName>
-        <imageTopicName>image_raw</imageTopicName>
-        <cameraInfoTopicName>camera_info</cameraInfoTopicName>
-        <frameName>camera</frameName>
-        <hackBaseline>0.07</hackBaseline>
-        <distortionK1>0.0</distortionK1>
-        <distortionK2>0.0</distortionK2>
-        <distortionK3>0.0</distortionK3>
-        <distortionT1>0.0</distortionT1>
-        <distortionT2>0.0</distortionT2>
-      </plugin>
-    </sensor>
-  </gazebo>
-  <link name="camera">
-    <visual>
-      <geometry>
-        <box size="0.05 0.05 0.05"/>
-      </geometry>
-    </visual>
-    <collision>
-      <geometry>
-        <box size="0.05 0.05 0.05"/>
-      </geometry>
-    </collision>
-    <xacro:default_inertial mass="0.02"/>
-  </link>
-  <joint name="camera_joint" type="fixed">
-    <origin xyz="0.73 0 1.18" rpy="0 0.45 0"/>
-    <parent link="body"/>
-    <child link="camera"/>
-  </joint>
+		<sensor type="camera" name="camera">
+		<update_rate>30.0</update_rate>
+			<camera name="head">
+				<horizontal_fov>1.3962634</horizontal_fov>
+				<image>
+				  <width>800</width>
+				  <height>800</height>
+				  <format>R8G8B8</format>
+				</image>
+				<clip>
+				  <near>0.02</near>
+				  <far>300</far>
+				</clip>
+				<noise>
+				  <type>gaussian</type>
+				  <mean>0.0</mean>
+				  <stddev>0.007</stddev>
+				</noise>
+			</camera>
+			<plugin name="camera_controller" filename="libgazebo_ros_camera.so">
+				<alwaysOn>true</alwaysOn>
+				<updateRate>0.0</updateRate>
+				<cameraName>/mybot/camera</cameraName>
+				<imageTopicName>image_raw</imageTopicName>
+				<cameraInfoTopicName>camera_info</cameraInfoTopicName>
+				<frameName>camera</frameName>
+				<hackBaseline>0.07</hackBaseline>
+				<distortionK1>0.0</distortionK1>
+				<distortionK2>0.0</distortionK2>
+				<distortionK3>0.0</distortionK3>
+				<distortionT1>0.0</distortionT1>
+				<distortionT2>0.0</distortionT2>
+			</plugin>
+		</sensor>
+	</gazebo>
+	<link name="camera">
+		<visual>
+			<geometry>
+				<box size="0.05 0.05 0.05"/>
+			</geometry>
+		</visual>
+		<collision>
+			<geometry>
+				<box size="0.05 0.05 0.05"/>
+			</geometry>
+		</collision>
+		<xacro:default_inertial mass="0.02"/>
+	</link>
+	<joint name="camera_joint" type="fixed">
+	<origin xyz="0.73 0 1.18" rpy="0 0.45 0"/>
+	<parent link="body"/>
+	<child link="camera"/>
+	</joint>
 </robot>

Commit message: made front wheel heavy to stop virat from lifting up

File: description/virat_description.urdf.xacro (robot description, xacro)
@@ -8,4 +8,18 @@
 		</inertial>
 	</xacro:macro>
+	<xacro:macro name="surface_coefficients">
+	 		<surface>
+				<bounce>
+					<restitution_coefficient>0.01</restitution_coefficient>
+					<threshold>0.5</threshold>
+				</bounce>
+        			<friction>
+        				<ode>
+        					<mu>100000</mu>
+        					<mu2>100000</mu2>
+        				</ode>
+        			</friction>
+        		</surface>
+        </xacro:macro>
 	<link name="base_link"/>
 	<link name="body">
@@ -41,12 +55,12 @@
 				<mesh filename="package://viratsim/meshes/wheels/castors1.dae"/>
         		</geometry>
-		</collision>
-		<xacro:default_inertial mass="1"/>
-	</link>
-	<joint name="front_axle" type="continuous">
+              		<xacro:surface_coefficients/>
+		</collision>
+		<xacro:default_inertial mass="15"/>
+	</link>
+	<joint name="front_axle" type="fixed">
 		<parent link="body"/>
 		<child link="front_wheel"/>
 		<origin xyz="0.48 0 0.02"/>
-		<axis xyz="0 1 0" rpy="0 0 0"/>
 	</joint>
 	<link name="rear_wheel_1">
@@ -62,4 +76,5 @@
 				<mesh filename="package://viratsim/meshes/wheels/tyre1.dae"/>
         		</geometry>
+        		<xacro:surface_coefficients/>
 		</collision>
 		<xacro:default_inertial mass="5"/>
@@ -70,4 +85,5 @@
 		<origin xyz="0 -0.323 0"/>
 		<axis xyz="0 1 0" rpy="0 0 0"/>
+		<joint_properties friction="100"/>
 	</joint>
 	<link name="rear_wheel_2">
@@ -83,4 +99,5 @@
 				<mesh filename="package://viratsim/meshes/wheels/tyre1.dae"/>
         		</geometry>
+        		<xacro:surface_coefficients/>
 		</collision>
 		<xacro:default_inertial mass="5"/>
@@ -91,4 +108,5 @@
 		<origin xyz="0 0.323 0"/>
 		<axis xyz="0 1 0" rpy="0 0 0"/>
+		<joint_properties friction="100"/>
 	</joint>
 	<gazebo reference="camera">
@@ -139,5 +157,5 @@
 			</geometry>
 		</collision>
-		<xacro:default_inertial mass="0.02"/>
+		<xacro:default_inertial mass="5"/>
 	</link>
 	<joint name="camera_joint" type="fixed">
@@ -146,16 +164,39 @@
 	<child link="camera"/>
 	</joint>
+	<gazebo>
 	<plugin name="differential_drive_controller" filename="libgazebo_ros_diff_drive.so">
- 		<alwaysOn>true</alwaysOn>
-		<updateRate>20</updateRate>
-		<leftJoint>rear_axle_2</leftJoint>
-		<rightJoint>rear_axle_1</rightJoint>
-		<wheelSeparation>0.323</wheelSeparation>
-		<wheelDiameter>0.04</wheelDiameter>
-		<torque>20</torque>
-		<commandTopic>/virat/cmd_vel</commandTopic>
-		<odometryTopic>/virat/odom</odometryTopic>
-		<odometryFrame>odom</odometryFrame>
-		<robotBaseFrame>body</robotBaseFrame>
- 	</plugin>
+	<!-- Plugin update rate in Hz -->
+	<updateRate>30</updateRate>
+	<!-- Name of left joint, defaults to `left_joint` -->
+	<leftJoint>rear_axle_1</leftJoint>
+	<!-- Name of right joint, defaults to `right_joint` -->
+	<rightJoint>rear_axle_2</rightJoint>
+	<!-- The distance from the center of one wheel to the other, in meters, defaults to 0.34 m -->
+	<wheelSeparation>0.646</wheelSeparation>
+	<!-- Diameter of the wheels, in meters, defaults to 0.15 m -->
+	<wheelDiameter>0.05</wheelDiameter>
+	<!-- Wheel acceleration, in rad/s^2, defaults to 0.0 rad/s^2 -->
+	<wheelAcceleration>1.0</wheelAcceleration>
+	<!-- Maximum torque which the wheels can produce, in Nm, defaults to 5 Nm -->
+	<wheelTorque>20</wheelTorque>
+	<!-- Topic to receive geometry_msgs/Twist message commands, defaults to `cmd_vel` -->
+	<commandTopic>cmd_vel</commandTopic>
+	<!-- Topic to publish nav_msgs/Odometry messages, defaults to `odom` -->
+	<odometryTopic>odom</odometryTopic>
+	<!-- Odometry frame, defaults to `odom` -->
+	<odometryFrame>odom</odometryFrame>
+	<!-- Robot frame to calculate odometry from, defaults to `base_footprint` -->
+	<robotBaseFrame>base_footprint</robotBaseFrame>
+	<!-- Odometry source, 0 for ENCODER, 1 for WORLD, defaults to WORLD -->
+	<odometrySource>1</odometrySource>
+	<!-- Set to true to publish transforms for the wheel links, defaults to false -->
+	<publishWheelTF>true</publishWheelTF>
+	<!-- Set to true to publish transforms for the odometry, defaults to true -->
+	<publishOdom>true</publishOdom>
+	<!-- Set to true to publish sensor_msgs/JointState on /joint_states for the wheel joints, defaults to false -->
+	<publishWheelJointState>true</publishWheelJointState>
+	<!-- Set to true to swap right and left wheels, defaults to true -->
+	<legacyMode>false</legacyMode>
+	</plugin>
+</gazebo>
 </robot>

Commit message: made mass variables for easy tweaking and made caster rotate about z to allow vehicle to turn

File: description/virat_description.urdf.xacro (robot description, xacro)
@@ -1,4 +1,8 @@
 <?xml version="1.0"?>
 <robot name="virat" xmlns:xacro="http://ros.org/wiki/xacro">
+	<xacro:property name="body_mass" value="50"/>
+	<xacro:property name="rear_wheel_mass" value="5"/>
+	<xacro:property name="castor_mass" value="15"/>
+	<xacro:property name="camera_mass" value="0.2"/>
 	<xacro:macro name="default_inertial" params="mass">
 		<inertial>
@@ -36,5 +40,5 @@
 			</geometry>
 		</collision>
-		<xacro:default_inertial mass="50"/>
+		<xacro:default_inertial mass="${body_mass}"/>
 	</link>
 	<joint name="dummy_joint" type="fixed">
@@ -57,10 +61,12 @@
               		<xacro:surface_coefficients/>
 		</collision>
-		<xacro:default_inertial mass="15"/>
-	</link>
-	<joint name="front_axle" type="fixed">
+		<xacro:default_inertial mass="${castor_mass}"/>
+	</link>
+	<joint name="front_axle" type="continuous">
 		<parent link="body"/>
 		<child link="front_wheel"/>
 		<origin xyz="0.48 0 0.02"/>
+		<axis xyz="0 0 1" rpy="0 0 0"/>
+		<joint_properties friction="100"/>
 	</joint>
 	<link name="rear_wheel_1">
@@ -78,5 +84,5 @@
         		<xacro:surface_coefficients/>
 		</collision>
-		<xacro:default_inertial mass="5"/>
+		<xacro:default_inertial mass="${rear_wheel_mass}"/>
 	</link>
 	<joint name="rear_axle_1" type="continuous">
@@ -101,5 +107,5 @@
         		<xacro:surface_coefficients/>
 		</collision>
-		<xacro:default_inertial mass="5"/>
+		<xacro:default_inertial mass="${rear_wheel_mass}"/>
 	</link>
 	<joint name="rear_axle_2" type="continuous">
@@ -157,5 +163,5 @@
 			</geometry>
 		</collision>
-		<xacro:default_inertial mass="5"/>
+		<xacro:default_inertial mass="${camera_mass}"/>
 	</link>
 	<joint name="camera_joint" type="fixed">

Commit message: Added camera feed, heavily modified teleop

File: description/virat_description.urdf.xacro (robot description, xacro)
@@ -9,5 +9,5 @@
 			<origin rpy="0.0 0 0" xyz="0 0 0"/>
 			<mass value="${mass}" />
-			<inertia ixx="1.0" ixy="0.0" ixz="0.0" iyy="1.0" iyz="0.0" izz="1.0" />
+			<inertia ixx="1" ixy="0.0" ixz="0.0" iyy="1" iyz="0.0" izz="1" />
 		</inertial>
 	</xacro:macro>
@@ -15,5 +15,5 @@
 	 		<surface>
 				<bounce>
-					<restitution_coefficient>0.01</restitution_coefficient>
+					<restitution_coefficient>0.00000000000000001</restitution_coefficient>
 					<threshold>0.5</threshold>
 				</bounce>
@@ -63,9 +63,8 @@
 		<xacro:default_inertial mass="${castor_mass}"/>
 	</link>
-	<joint name="front_axle" type="continuous">
+	<joint name="front_axle" type="fixed">
 		<parent link="body"/>
 		<child link="front_wheel"/>
 		<origin xyz="0.48 0 0.02"/>
-		<axis xyz="0 0 1" rpy="0 0 0"/>
 		<joint_properties friction="100"/>
 	</joint>

Commit message: Final commit. Project complete.

File: description/virat_description.urdf.xacro (robot description, xacro)
@@ -20,6 +20,6 @@
         			<friction>
         				<ode>
-        					<mu>100000</mu>
-        					<mu2>100000</mu2>
+        					<mu>100000000000</mu>
+        					<mu2>100000000000</mu2>
         				</ode>
         			</friction>
@@ -27,4 +27,10 @@
         </xacro:macro>
 	<link name="base_link"/>
+	<link name="odom"/>
+	<joint name="odom_joint" type="fixed">
+		<parent link="base_link"/>
+		<child link="odom"/>
+		<origin xyz="0 0 0"/>
+	</joint>
 	<link name="body">
 		<visual>
@@ -165,7 +171,7 @@
 	</link>
 	<joint name="camera_joint" type="fixed">
-	<origin xyz="0.73 0 1.18" rpy="0 0.45 0"/>
-	<parent link="body"/>
-	<child link="camera"/>
+		<origin xyz="0.73 0 1.18" rpy="0 0.45 0"/>
+		<parent link="base_link"/>
+		<child link="camera"/>
 	</joint>
 	<gazebo>

Commit message: removed redundant transforms; tf not fixed fully tho

File: description/virat_description.urdf.xacro (robot description, xacro)
@@ -27,10 +27,4 @@
         </xacro:macro>
 	<link name="base_link"/>
-	<link name="odom"/>
-	<joint name="odom_joint" type="fixed">
-		<parent link="base_link"/>
-		<child link="odom"/>
-		<origin xyz="0 0 0"/>
-	</joint>
 	<link name="body">
 		<visual>
@@ -188,7 +182,6 @@
 	<odometryFrame>odom</odometryFrame>
 	<robotBaseFrame>base_footprint</robotBaseFrame>
-	<odometrySource>1</odometrySource>
-	<publishWheelTF>true</publishWheelTF>
-	<publishOdom>true</publishOdom>
+	<publishOdomTF>true</publishOdomTF>
+	<publishWheelTF>false</publishWheelTF>
 	<publishWheelJointState>true</publishWheelJointState>
 	<legacyMode>false</legacyMode>
